Commit message: Fix dual arm simulation and test the YMCA mission director

File: src/simulation/px4_uam_sim/urdf/martijn.xacro (robot description, xacro)
@@ -212,5 +212,5 @@
     <parent link="base_link"/>
     <child link="shoulder_link_1"/>
-    <origin xyz="0.015 0 0" rpy="1.5708 0 -1.5708"/>
+    <origin xyz="0.015 0 0" rpy="1.5708 -1.5708 -1.5708"/>
     <axis xyz="0 0 -1"/>
     <limit lower="-6.28" upper="6.28" velocity="2.0" effort="100.0"/>
@@ -274,6 +274,6 @@
     <parent link="motor_link_shoulder_1"/>
     <child link="elbow_link_1"/>
-    <origin xyz="0 0 0.0125" rpy="1.5708 1.5708 0"/>
-    <axis xyz="0 0 -1"/>
+    <origin xyz="0 0 0.0125" rpy="1.5708 1.5708 3.14"/>
+    <axis xyz="0 0 1"/>
     <limit lower="-1.5708" upper="1.5708" velocity="2" effort="100"/>
     <dynamics damping="0.01" friction="0.1"/>
@@ -338,5 +338,5 @@
     <origin xyz="-0.31 0 0" rpy="0 0 0"/>
     <axis xyz="0 -1 0"/>
-    <limit lower="-1.5708" upper="1.9" velocity="20" effort="100"/>
+    <limit lower="-1.9" upper="1.9" velocity="20" effort="100"/>
     <dynamics damping="0.0001" friction="0.0"/>
   </joint>
@@ -369,5 +369,5 @@
     <parent link="base_link"/>
     <child link="shoulder_link_2"/>
-    <origin xyz="-0.015 0 0" rpy="1.5708 0 1.5708"/>
+    <origin xyz="-0.015 0 0" rpy="1.5708 -1.5708 1.5708"/>
     <axis xyz="0 0 1"/>
     <limit lower="-6.28" upper="6.28" velocity="2.0" effort="100.0"/>
@@ -406,5 +406,5 @@
   <link name="elbow_link_2">
     <collision>
-      <origin xyz="-0.16 0 0" rpy="0 0 0"/>
+      <origin xyz="-0.16 0 0" rpy="0 0 3.14"/>
       <geometry>
         <box size="0.34 0.024 0.054"/>
@@ -495,5 +495,5 @@
     <origin xyz="-0.31 0 0" rpy="0 0 0"/>
     <axis xyz="0 -1 0"/>
-    <limit lower="-1.5708" upper="1.9" velocity="20" effort="100"/>
+    <limit lower="-1.9" upper="1.9" velocity="20" effort="100"/>
     <dynamics damping="0.0001" friction="0.0"/>
   </joint>
